File: hard/avr/pro_mini/avr_saber_mini.brd (EAGLE design)
At the start: 83.5 x 34.3 mm, 32 parts, among them U3 USD-SOCKETUSD

Commit message: correction inhibit pth
Connections:
- net GND: no longer U$4.5
Changed lines of the file:
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@@
 <contactref element="C8" pad="2"/>
 <contactref element="C5" pad="2"/>
-<contactref element="U$4" pad="5"/>
 <contactref element="U1" pad="11"/>
 <contactref element="MMA8451" pad="GND"/>
