File: hard/avr/pro_mini/avr_saber_mini.brd (EAGLE design)
At the start: 83.5 x 34.3 mm, 32 parts, among them U3 USD-SOCKETUSD

Commit message: ajout de la dernière version de carte
Parts:
- moved ADC1 1.82 mm to (42.5, 5.89)
- moved R12 0.81 mm to (76.5, 26.8), turned to 270 degrees
- moved R9 0.41 mm to (76.2, 23.5)
Connections:
- net +5V: now also R11.1
- net GND: no longer R11.1
Routing:
- net +5V: track 147.4 -> 156.6 mm
- net N$7: track 17.1 -> 25.8 mm
- net MOSI: track 33.3 -> 26.3 mm
- net DAC_LATCH: track 24.6 -> 21.1 mm
- net N$32: track 8.03 -> 11.5 mm
- net SCK: track 18.9 -> 22.2 mm, vias 1 -> 2
- net GND: track 5.15 -> 8.39 mm
- net N$33: track 5.26 -> 7.11 mm
- net MISO: track 22.5 -> 21.0 mm, vias 1 -> 2
- net N$4: track 3.19 -> 4.57 mm
- net N$17: track 3.19 -> 4.53 mm
- net N$16: track 3.19 -> 4.53 mm
- net N$14: track 3.19 -> 4.53 mm
- net +3V3: track 127.3 -> 128.0 mm
