File: hard/avr/pro_mini/avr_saber_mini_v2.brd (EAGLE design)
At the start: 83.5 x 34.3 mm, 32 parts, among them U3 USD-SOCKETUSD

Commit message: ajout divers soft
Connections:
- net +5V: now also U$1.SHUTDOWN
Changed lines of the file:
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@@
 <contactref element="U$5" pad="3"/>
 <contactref element="C9" pad="2"/>
-<wire x1="-8.8036" y1="-45.1104" x2="-16.764" y2="-40.1454" width="0" layer="19" extent="1-1"/>
-<wire x1="36.83" y1="6.35" x2="-8.8036" y2="-45.1104" width="0" layer="19" extent="1-1"/>
-<wire x1="42.3164" y1="3.8608" x2="42.2148" y2="3.7592" width="0" layer="19" extent="1-1"/>
+<contactref element="U$1" pad="SHUTDOWN"/>
+<wire x1="71.4756" y1="24.4856" x2="72.1082" y2="24.4938" width="0" layer="19" extent="16-16"/>
+<wire x1="42.2148" y1="3.7592" x2="42.3164" y2="3.8608" width="0" layer="19" extent="1-1"/>
+<wire x1="-8.8036" y1="-45.1104" x2="36.83" y2="6.35" width="0" layer="19" extent="1-1"/>
+<wire x1="-16.764" y1="-40.1454" x2="-8.8036" y2="-45.1104" width="0" layer="19" extent="1-1"/>
 </signal>
 <signal name="GND">
