File: hard/avr/pro_mini/avr_saber_mini_v2.brd (EAGLE design)
At the start: 83.5 x 34.3 mm, 32 parts, among them U3 USD-SOCKETUSD

Commit message: no
Parts:
- added HP_SECOURS: (no value), pinhead:1X02
- moved R13 90.4 mm to (62.0, 6.91), turned to 90 degrees
- moved C10 85.0 mm to (20.5, 16.1), turned to 90 degrees
- moved R8 81.4 mm to (56.1, 6.30), flipped to the bottom, turned to 90 degrees
- moved R10 78.1 mm to (51.2, 6.30), flipped to the bottom, turned to 90 degrees
- moved R1 78.0 mm to (53.6, 6.30), flipped to the bottom, turned to 90 degrees
- moved C9 77.2 mm to (21.7, 25.4), turned to 180 degrees
- moved U$5 58.1 mm to (5.69, 22.6), turned to 90 degrees
- moved R3 7.34 mm to (11.5, 7.85), turned to 90 degrees
- moved R2 5.08 mm to (7.87, 10.2)
- moved BLUETOOTH 1.63 mm to (28.7, 29.4)
- moved C2 1.29 mm to (22.7, 29.9)
- moved HP 0.61 mm to (72.0, 31.2)
Connections:
- net +5V: now also U$1.SHUTDOWN
- net GND: now also HP_SECOURS.2
- net N$15: now also HP_SECOURS.1
Routing:
- net N$9: track 13.9 -> 49.0 mm
- net N$11: track 13.9 -> 41.0 mm, vias 0 -> 1
- net GND: track 1.03 -> 26.3 mm
- net N$7: track 17.0 -> 41.0 mm, vias 2 -> 1
- net MOSI: track 25.6 -> 2.65 mm, vias 1 -> 0
- net MISO: track 24.0 -> 2.69 mm, vias 1 -> 0
- net MMC_CS: track 23.0 -> 4.00 mm
- net N$6: track 20.9 -> 38.7 mm, vias 2 -> 1
- net SCK: track 18.8 -> 2.73 mm, vias 1 -> 0
- net +12V: track 45.7 -> 59.5 mm, vias 0 -> 1
- net N$15: track 18.5 -> 26.6 mm
- net +5V: track 144.0 -> 149.4 mm, vias 2 -> 3
- net N$1: track 0.00 -> 4.06 mm
- net DAC_LATCH: track 24.6 -> 27.9 mm
- net BATTLEVEL: track 72.7 -> 69.7 mm, vias 1 -> 0
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Other:
- board text added: "3V3"
- board text added: "5V"
- board text added: "ADC"
- board text added: "BAT"
- board text added: "HP"
- board text added: "LED"
