File: hard/avr/pro_mini/avr_saber_mini_v2.sch (EAGLE design)
At the start: 32 parts, among them U3 USD-SOCKETUSD

Commit message: ajout divers soft
Connections:
- net +5V: now also U$1.|SHUTDOWN
Changed lines of the file:
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@@
 <wire x1="195.58" y1="139.7" x2="193.04" y2="139.7" width="0.1524" layer="91"/>
 <wire x1="195.58" y1="139.7" x2="195.58" y2="144.78" width="0.1524" layer="91"/>
+<pinref part="U$1" gate="G$1" pin="|SHUTDOWN"/>
+<wire x1="198.12" y1="144.78" x2="182.88" y2="144.78" width="0.1524" layer="91"/>
+<wire x1="175.26" y1="144.78" x2="182.88" y2="144.78" width="0.1524" layer="91"/>
+<wire x1="182.88" y1="144.78" x2="182.88" y2="137.16" width="0.1524" layer="91"/>
+<wire x1="182.88" y1="137.16" x2="198.12" y2="137.16" width="0.1524" layer="91"/>
+<wire x1="198.12" y1="137.16" x2="198.12" y2="139.7" width="0.1524" layer="91"/>
 </segment>
 <segment>
