File: hard/avr/pro_mini/avr_saber_mini.sch (EAGLE design)
At the start: 32 parts, among them U3 USD-SOCKETUSD

Commit message: correction inhibit pth
Connections:
- net GND: no longer U$4.INH
Changed lines of the file:
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@@
 <?xml version="1.0" encoding="utf-8"?>
 <!DOCTYPE eagle SYSTEM "eagle.dtd">
-<eagle version="6.4">
+<eagle version="6.5.0">
 <drawing>
 <settings>
@@
 <wire x1="-35.56" y1="111.76" x2="-48.26" y2="111.76" width="0.1524" layer="91"/>
 <pinref part="C8" gate="G$1" pin="2"/>
-<wire x1="-63.5" y1="111.76" x2="-55.88" y2="111.76" width="0.1524" layer="91"/>
 <pinref part="C5" gate="G$1" pin="2"/>
-<wire x1="-55.88" y1="111.76" x2="-48.26" y2="111.76" width="0.1524" layer="91"/>
+<wire x1="-63.5" y1="111.76" x2="-48.26" y2="111.76" width="0.1524" layer="91"/>
 <wire x1="-27.94" y1="121.92" x2="-27.94" y2="111.76" width="0.1524" layer="91"/>
 <wire x1="-27.94" y1="111.76" x2="-35.56" y2="111.76" width="0.1524" layer="91"/>
-<pinref part="U$4" gate="G$1" pin="INH"/>
-<wire x1="-55.88" y1="121.92" x2="-55.88" y2="111.76" width="0.1524" layer="91"/>
-<junction x="-55.88" y="111.76"/>
 <junction x="-48.26" y="111.76"/>
 <junction x="-35.56" y="111.76"/>

Commit message: ajout de la dernière version de carte
Connections:
- net +5V: now also R11.1
- net GND: no longer R11.1
Changed lines of the file:
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@@
 <part name="GND25" library="supply2" deviceset="GND" device=""/>
 <part name="R11" library="rcl" deviceset="R-EU_" device="R0805"/>
-<part name="GND26" library="supply2" deviceset="GND" device=""/>
 <part name="HP" library="pinhead" deviceset="PINHD-1X2" device=""/>
 <part name="R12" library="rcl" deviceset="R-EU_" device="R0805"/>
@@
 <part name="GND24" library="supply1" deviceset="GND" device=""/>
 <part name="+3V4" library="supply1" deviceset="+3V3" device=""/>
+<part name="P+1" library="supply1" deviceset="+5V" device=""/>
 </parts>
 <sheets>
@@
 <instance part="GND25" gate="GND" x="193.04" y="124.46"/>
 <instance part="R11" gate="G$1" x="175.26" y="139.7" rot="R90"/>
-<instance part="GND26" gate="GND" x="175.26" y="132.08"/>
 <instance part="HP" gate="G$1" x="284.48" y="142.24"/>
 <instance part="R12" gate="G$1" x="251.46" y="144.78"/>
@@
 <instance part="GND24" gate="1" x="73.66" y="68.58" rot="R90"/>
 <instance part="+3V4" gate="G$1" x="-25.4" y="-27.94" rot="R90"/>
+<instance part="P+1" gate="1" x="165.1" y="142.24"/>
 </instances>
 <busses>
@@
 <wire x1="73.66" y1="71.12" x2="71.12" y2="71.12" width="0.1524" layer="91"/>
 </segment>
+<segment>
+<pinref part="P+1" gate="1" pin="+5V"/>
+<wire x1="165.1" y1="139.7" x2="165.1" y2="132.08" width="0.1524" layer="91"/>
+<pinref part="R11" gate="G$1" pin="1"/>
+<wire x1="165.1" y1="132.08" x2="175.26" y2="132.08" width="0.1524" layer="91"/>
+<wire x1="175.26" y1="132.08" x2="175.26" y2="134.62" width="0.1524" layer="91"/>
+</segment>
 </net>
 <net name="GND" class="0">
@@
 </segment>
 <segment>
-<pinref part="R11" gate="G$1" pin="1"/>
-<pinref part="GND26" gate="GND" pin="GND"/>
-</segment>
-<segment>
