File: hard/led/led_saber.brd (EAGLE design)
At the start: 26.3 x 24.1 mm, 5 parts, among them IC2 CAT4101

Commit message: ajout readme divers
Parts:
- moved R2 1.78 mm to (7.98, 4.06)
- moved LED 0.91 mm to (17.8, 3.45)
Routing:
- net GND: track 11.4 -> 4.35 mm
- net N$1: track 16.8 -> 22.5 mm
- net PWM: track 6.30 -> 3.96 mm
- net N$2: track 6.51 -> 7.71 mm
- net +5V: track 5.13 -> 3.96 mm
Other:
- board size 26.3 x 24.1 mm -> 24.1 x 22.9 mm
- board text added: "LightsaberEnsea"
Changed lines of the file:
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@@
 <grid distance="0.025" unitdist="inch" unit="inch" style="lines" multiple="1" display="yes" altdistance="0.025" altunitdist="inch" altunit="inch"/>
 <layers>
-<layer number="1" name="Top" color="4" fill="1" visible="no" active="yes"/>
+<layer number="1" name="Top" color="4" fill="1" visible="yes" active="yes"/>
 <layer number="16" name="Bottom" color="1" fill="1" visible="yes" active="yes"/>
 <layer number="17" name="Pads" color="2" fill="1" visible="yes" active="yes"/>
@@
 <layer number="19" name="Unrouted" color="6" fill="1" visible="yes" active="yes"/>
 <layer number="20" name="Dimension" color="15" fill="1" visible="yes" active="yes"/>
-<layer number="21" name="tPlace" color="7" fill="1" visible="no" active="yes"/>
-<layer number="22" name="bPlace" color="7" fill="1" visible="no" active="yes"/>
-<layer number="23" name="tOrigins" color="15" fill="1" visible="no" active="yes"/>
-<layer number="24" name="bOrigins" color="15" fill="1" visible="no" active="yes"/>
+<layer number="21" name="tPlace" color="7" fill="1" visible="yes" active="yes"/>
+<layer number="22" name="bPlace" color="7" fill="1" visible="yes" active="yes"/>
+<layer number="23" name="tOrigins" color="15" fill="1" visible="yes" active="yes"/>
+<layer number="24" name="bOrigins" color="15" fill="1" visible="yes" active="yes"/>
 <layer number="25" name="tNames" color="7" fill="1" visible="no" active="yes"/>
 <layer number="26" name="bNames" color="7" fill="1" visible="no" active="yes"/>
@@
 <board>
 <plain>
-<wire x1="0" y1="0" x2="26.34" y2="0" width="0" layer="20"/>
-<wire x1="26.34" y1="0" x2="26.34" y2="24.12" width="0" layer="20"/>
-<wire x1="26.34" y1="24.12" x2="0" y2="24.12" width="0" layer="20"/>
-<wire x1="0" y1="24.12" x2="0" y2="0" width="0" layer="20"/>
-<text x="10.16" y="4.445" size="1.016" layer="1" font="vector" ratio="12">GND/+5V/D</text>
+<text x="10.795" y="5.08" size="1.016" layer="1" font="vector" ratio="12">GND/+5V/D</text>
 <text x="4.445" y="13.335" size="1.27" layer="1" ratio="13" rot="R90">Vled+</text>
 <text x="9.525" y="6.985" size="1.016" layer="1" ratio="13">Lightsaber C&amp;T</text>
-<text x="1.27" y="1.27" size="1.016" layer="16" ratio="13" rot="MR90">Lightsaber C&amp;T</text>
+<text x="24.4348" y="10.1092" size="0.8128" layer="16" font="vector" ratio="12" rot="MR295">Lightsaber C&amp;T</text>
+<wire x1="6.35" y1="0" x2="20.32" y2="0" width="0.3048" layer="20"/>
+<wire x1="20.32" y1="0" x2="25.4" y2="5.08" width="0.3048" layer="20"/>
+<wire x1="25.4" y1="5.08" x2="25.4" y2="17.78" width="0.3048" layer="20"/>
+<wire x1="25.4" y1="17.78" x2="20.32" y2="22.86" width="0.3048" layer="20"/>
+<wire x1="20.32" y1="22.86" x2="6.35" y2="22.86" width="0.3048" layer="20"/>
+<wire x1="6.35" y1="22.86" x2="1.27" y2="17.78" width="0.3048" layer="20"/>
+<wire x1="1.27" y1="17.78" x2="1.27" y2="5.08" width="0.3048" layer="20"/>
+<wire x1="1.27" y1="5.08" x2="6.35" y2="0" width="0.3048" layer="20"/>
+<text x="6.985" y="19.685" size="1.016" layer="1" font="vector" ratio="12">LightsaberEnsea</text>
 </plain>
 <attributes>
@@
 <attribute name="OC_FARNELL" value="1718452" x="-5.08" y="5.08" size="1.778" layer="28" rot="MR0" display="off"/>
 </element>
-<element name="R2" library="resistor" package="R0805" value="549" x="8.89" y="2.54" rot="MR90"/>
-<element name="LED" library="SparkFun-Electromechanical" package="1X03" value="SMALL_SERVO" x="17.78" y="2.54" rot="R180"/>
+<element name="R2" library="resistor" package="R0805" value="549" x="7.9756" y="4.064" rot="MR90"/>
+<element name="LED" library="SparkFun-Electromechanical" package="1X03" value="SMALL_SERVO" x="17.78" y="3.4544" rot="R180"/>
 <element name="LED1" library="led" package="Z-POWER-LED-DOME-TYPE" value="X42182" x="13.97" y="12.7"/>
 <element name="VBAT" library="SparkFun-Connectors" package="1X01" value="M01PTH" x="4.445" y="11.43"/>
@@
 <contactref element="LED" pad="3"/>
 <polygon width="0.4064" layer="16" isolate="0.6096">
-<vertex x="0" y="29.21"/>
+<vertex x="-2.1336" y="29.5148"/>
 <vertex x="29.21" y="29.21"/>
-<vertex x="29.21" y="0"/>
-<vertex x="0" y="0"/>
+<vertex x="30.4292" y="-4.8768"/>
+<vertex x="-3.048" y="-4.572"/>
 </polygon>
 <polygon width="0.4064" layer="1" isolate="0.6096">
-<vertex x="-2.54" y="31.75"/>
-<vertex x="-2.54" y="-2.54"/>
-<vertex x="33.02" y="-2.54"/>
+<vertex x="-7.7216" y="31.4452"/>
+<vertex x="-7.7216" y="-6.5024"/>
+<vertex x="33.02" y="-6.1976"/>
 <vertex x="33.02" y="31.75"/>
 </polygon>
-<wire x1="12.7" y1="2.54" x2="12.7" y2="3.81" width="1.016" layer="16"/>
-<wire x1="12.7" y1="3.81" x2="13.97" y2="5.08" width="1.016" layer="16"/>
-<wire x1="13.97" y1="5.08" x2="13.97" y2="7.24" width="1.016" layer="16"/>
-<wire x1="13.97" y1="8.89" x2="13.97" y2="7.24" width="1.016" layer="16"/>
-<wire x1="12.7" y1="2.54" x2="11.43" y2="1.27" width="1.016" layer="16"/>
-<wire x1="11.43" y1="1.27" x2="9.31" y2="1.27" width="1.016" layer="16"/>
-<wire x1="9.31" y1="1.27" x2="8.89" y2="1.69" width="1.016" layer="16"/>
+<wire x1="12.7" y1="3.4544" x2="12.7" y2="4.1656" width="0.6096" layer="16"/>
+<wire x1="12.7" y1="4.1656" x2="14.0208" y2="5.4864" width="0.6096" layer="16"/>
+<wire x1="14.0208" y1="5.4864" x2="14.0208" y2="7.1892" width="0.6096" layer="16"/>
+<wire x1="14.0208" y1="7.1892" x2="13.97" y2="7.24" width="0.6096" layer="16"/>
 </signal>
 <signal name="N$2">
 <contactref element="R2" pad="2"/>
 <contactref element="IC2" pad="4"/>
-<wire x1="8.89" y1="3.39" x2="9.74" y2="3.39" width="0.6096" layer="16"/>
-<wire x1="9.74" y1="3.39" x2="12.065" y2="5.715" width="0.6096" layer="16"/>
-<wire x1="12.065" y1="5.715" x2="12.065" y2="7.62" width="0.6096" layer="16"/>
-<wire x1="12.27" y1="7.24" x2="12.27" y2="7.415" width="0.6096" layer="16"/>
-<wire x1="12.27" y1="7.415" x2="12.065" y2="7.62" width="0.6096" layer="16"/>
+<wire x1="7.9756" y1="4.914" x2="11.2404" y2="4.914" width="0.6096" layer="16"/>
+<wire x1="11.2404" y1="4.914" x2="11.2776" y2="4.8768" width="0.6096" layer="16"/>
+<wire x1="11.2776" y1="4.8768" x2="12.4968" y2="6.096" width="0.6096" layer="16"/>
+<wire x1="12.4968" y1="6.096" x2="12.4968" y2="7.62" width="0.6096" layer="16"/>
+<wire x1="12.4968" y1="7.62" x2="12.192" y2="7.9248" width="0.6096" layer="16"/>
+<wire x1="12.192" y1="7.9248" x2="12.192" y2="7.318" width="0.6096" layer="16"/>
+<wire x1="12.192" y1="7.318" x2="12.27" y2="7.24" width="0.6096" layer="16"/>
 </signal>
 <signal name="PWM">
 <contactref element="IC2" pad="1"/>
 <contactref element="LED" pad="1"/>
-<wire x1="17.78" y1="2.54" x2="17.78" y2="6.35" width="1.016" layer="16"/>
-<wire x1="17.78" y1="6.35" x2="17.145" y2="6.985" width="1.016" layer="16"/>
-<wire x1="17.145" y1="6.985" x2="17.145" y2="7.465" width="1.016" layer="16"/>
-<wire x1="17.145" y1="8.255" x2="17.145" y2="7.465" width="1.016" layer="16"/>
-<wire x1="17.145" y1="7.465" x2="17.37" y2="7.24" width="1.016" layer="16"/>
+<wire x1="17.78" y1="3.4544" x2="17.78" y2="5.08" width="0.6096" layer="16"/>
+<wire x1="17.78" y1="5.08" x2="17.3736" y2="5.4864" width="0.6096" layer="16"/>
+<wire x1="17.3736" y1="5.4864" x2="17.3736" y2="7.2364" width="0.6096" layer="16"/>
+<wire x1="17.3736" y1="7.2364" x2="17.37" y2="7.24" width="0.6096" layer="16"/>
 </signal>
 <signal name="+5V">
 <contactref element="LED" pad="2"/>
 <contactref element="IC2" pad="2"/>
-<wire x1="15.24" y1="2.54" x2="15.67" y2="2.54" width="1.016" layer="16"/>
-<wire x1="15.67" y1="2.54" x2="15.67" y2="7.24" width="1.016" layer="16"/>
+<wire x1="15.24" y1="3.4544" x2="15.24" y2="4.572" width="0.6096" layer="16"/>
+<wire x1="15.24" y1="4.572" x2="15.5448" y2="4.8768" width="0.6096" layer="16"/>
+<wire x1="15.5448" y1="4.8768" x2="15.5448" y2="7.1148" width="0.6096" layer="16"/>
+<wire x1="15.5448" y1="7.1148" x2="15.67" y2="7.24" width="0.6096" layer="16"/>
 </signal>
 <signal name="N$1">
 <contactref element="IC2" pad="5"/>
 <contactref element="LED1" pad="C"/>
-<wire x1="10.57" y1="7.24" x2="10.57" y2="10.57" width="1.016" layer="16"/>
-<wire x1="10.57" y1="10.57" x2="11.43" y2="11.43" width="1.016" layer="16"/>
-<wire x1="11.43" y1="11.43" x2="19.685" y2="11.43" width="1.016" layer="16"/>
-<wire x1="19.685" y1="11.43" x2="20.32" y2="10.795" width="1.016" layer="16"/>
-<via x="20.32" y="10.795" extent="1-16" drill="1.2"/>
-<wire x1="20.62" y1="13.82" x2="20.62" y2="11.095" width="1.016" layer="1"/>
-<wire x1="20.62" y1="11.095" x2="20.32" y2="10.795" width="1.016" layer="1"/>
+<wire x1="10.57" y1="7.24" x2="10.668" y2="7.24" width="1.016" layer="16"/>
+<wire x1="10.668" y1="7.24" x2="10.668" y2="10.720296875" width="1.016" layer="16"/>
+<wire x1="10.668" y1="10.720296875" x2="11.530103125" y2="11.5824" width="1.016" layer="16"/>
+<wire x1="11.530103125" y1="11.5824" x2="23.115340625" y2="11.5824" width="1.016" layer="16"/>
+<wire x1="23.115340625" y1="11.5824" x2="24.0792" y2="12.546259375" width="1.016" layer="16"/>
+<wire x1="24.0792" y1="12.546259375" x2="24.0792" y2="13.716" width="1.016" layer="16"/>
+<via x="24.0792" y="13.716" extent="1-16" drill="1.2"/>
+<wire x1="24.0792" y1="13.716" x2="20.62" y2="13.716" width="1.016" layer="1"/>
+<wire x1="20.62" y1="13.716" x2="20.62" y2="13.82" width="1.016" layer="1"/>
 </signal>
 <signal name="N$3">
